File: Atmega328p-DevBoard-Hardware.kicad_sch (KiCad schematic)
At the start: 0 parts

Commit message: completed power supply design section with schematics, now working on MCU Section
Parts:
- added C1, C3: 100uf, 25V, Capacitor_SMD:C_Elec_6.3x7.7, symbol Device:C_Small_US
- added C2, C4, C5, C6, C7: 0.1uf, Capacitor_SMD:C_0805_2012Metric_Pad1.18x1.45mm_HandSolder, symbol Device:C_Small
- added C8: 22uf, Capacitor_SMD:C_0805_2012Metric_Pad1.18x1.45mm_HandSolder, symbol Device:C_Small
- added D1: SS14 (1A,40V), Diode_SMD:D_SMA_Handsoldering, symbol Device:D_Schottky
- added D2: RLED, LED_SMD:LED_0805_2012Metric_Pad1.15x1.40mm_HandSolder, symbol Device:LED
- added J1: Barrel_Jack, Connector_BarrelJack:BarrelJack_Horizontal, symbol Connector:Barrel_Jack_MountingPin
- added R1: 220, Resistor_SMD:R_0805_2012Metric_Pad1.20x1.40mm_HandSolder, symbol Device:R_Small_US
- added U1: L7805, Package_TO_SOT_SMD:TO-252-2, symbol Regulator_Linear:L7805
- added U2: ATmega328P-A, Package_QFP:TQFP-32_7x7mm_P0.8mm, symbol MCU_Microchip_ATmega:ATmega328P-A
Connections:
- new net: D2.2 (A), R1.2
- new net: D1.2 (A), J1.1
- new net +12V: C1.1, C2.1, D1.1 (K), U1.1 (IN)
- new net +5V: C3.1, C4.1, C5.1, C6.1, C7.1, C8.1, R1.1, U1.3 (OUT), U2.18 (AVCC), U2.4 (VCC), U2.6 (VCC)
- new net GND: C1.2, C2.2, C3.2, C4.2, C5.2, C6.2, C7.2, C8.2, D2.1 (K), J1.2, J1.MP (MountPin), U1.2 (GND), U2.21 (GND), U2.3 (GND), U2.5 (GND)
Other:
- note added: "Note: 1. 2 Vcc pins & 1 AVcc pins 2. Filtering for each Vcc and VAcc pin 3. Bulk Capacitor for MCU's Quick Current consumption requirements"
- title: (none) -> ATMEGA328p Dev Board

Commit message: finished motor driver design section in docs and schematics
Parts:
- added C10, C11, C12, C15, C9: 0.1uf, Capacitor_SMD:C_0805_2012Metric_Pad1.18x1.45mm_HandSolder, symbol Device:C_Small
- added C13: 10uf, Capacitor_SMD:C_0805_2012Metric_Pad1.18x1.45mm_HandSolder, symbol Device:C_Small
- added C14: 100uf, Capacitor_SMD:C_0805_2012Metric_Pad1.18x1.45mm_HandSolder, symbol Device:C_Small
- added J2: DBG/PROG, Connector_PinSocket_2.54mm:PinSocket_2x04_P2.54mm_Vertical, symbol Connector_Generic:Conn_02x04_Odd_Even
- added J3: MTR1-CON, Connector_Phoenix_MC:PhoenixContact_MC_1,5_2-G-3.81_1x02_P3.81mm_Horizontal, symbol Connector:Conn_01x02_Pin
- added J4: MTR2-CON, Connector_Phoenix_MC:PhoenixContact_MC_1,5_2-G-3.81_1x02_P3.81mm_Horizontal, symbol Connector:Conn_01x02_Pin
- added R2: 10K, Resistor_SMD:R_0805_2012Metric_Pad1.20x1.40mm_HandSolder, symbol Device:R_Small_US
- added SW1: SW_SPST, Button_Switch_THT:SW_PUSH_6mm, symbol Switch:SW_SPST
- added U3: L293D, Package_DIP:DIP-16_W7.62mm, symbol Driver_Motor:L293D
- added Y1: LFXTAL003237-Crystal-16MHz, Crystal:Crystal_SMD_HC49-SD_HandSoldering, symbol Device:Crystal
- R1: value 220 -> 10K
Connections:
- net +12V: now also C14.1, C15.1, U3.8 (VCC2)
- net +5V: now also C12.1, C13.1, J2.7 (Pin_7), R2.1, U3.16 (VCC1)
- net GND: now also C10.1, C11.1, C12.2, C13.2, C14.2, C15.2, C9.2, J2.8 (Pin_8), SW1.1 (A), U3.12 (GND), U3.13 (GND), U3.4 (GND), U3.5 (GND)
- net MTR2_DIR1: now reaches U2.10 (PD6)
- net MTR2_DIR1: now also U3.10 (3A)
- net MTR2_DIR2: now reaches U2.11 (PD7)
- net MTR2_DIR2: now also U3.15 (4A)
- net MTR1_DIR2: now reaches U2.12 (PB0)
- net MTR1_DIR2: now also U3.7 (2A)
- net MTR1_PWM: now reaches U2.13 (PB1)
- net MTR1_PWM: now also U3.1 (EN1,2)
- net MTR2_PWM: now reaches U2.14 (PB2)
- net MTR2_PWM: now also U3.9 (EN3,4)
- net MOSI: now reaches U2.15 (PB3)
- net MOSI: now also J2.2 (Pin_2)
- net MISO: now reaches U2.16 (PB4)
- net MISO: now also J2.1 (Pin_1)
- net SCK: now reaches U2.17 (PB5)
- net SCK: now also J2.4 (Pin_4)
- net RESET: now reaches U2.29 (~{RESET}/PC6)
- net RESET: now also C9.1, J2.3 (Pin_3), R2.2, SW1.2 (B)
- net DEBUG_RXD: now reaches U2.30 (PD0)
- net DEBUG_RXD: now also J2.5 (Pin_5)
- net DEBUG_TXD: now reaches U2.31 (PD1)
- net DEBUG_TXD: now also J2.6 (Pin_6)
- net XTAL1: now reaches U2.7 (XTAL1/PB6)
- net XTAL1: now also C10.2, Y1.1
- net XTAL2: now reaches U2.8 (XTAL2/PB7)
- net XTAL2: now also C11.2, Y1.2
- net MTR1_DIR1: now reaches U2.9 (PD5)
- net MTR1_DIR1: now also U3.2 (1A)
- new net: J3.1 (Pin_1), U3.3 (1Y)
- new net: J3.2 (Pin_2), U3.6 (2Y)
- new net: J4.1 (Pin_1), U3.11 (3Y)
- new net: J4.2 (Pin_2), U3.14 (4Y)
Other:
- note added: "ATMEGA328P BASED DEVELOPMENT BOARD DESIGN"
- note added: "Debug/Program Interface"
- note added: "External Oscillator"
- note added: "MCU PWR Rail Input Filtering"
- note added: "Reset Switch"
- moved on the sheet: C1, C2, C3, C4, C5, C6, C7, C8, D1, D2, J1, R1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
